Commit message: Use validated Allen key manipulation grasps

File: assets/urdf/workpieces/allen_key_hex_socket.urdf (robot description, URDF)
Before this commit: robot allen_key_hex_socket, 1 links, 0 joints
Links:
- link workpiece_root: geometry collision box size=0.008 0.020 0.025; collision box size=0.008 0.020 0.025
