Commit message: Remake Allen key with thin hex profile

File: assets/urdf/objects/allen_key_canonical.urdf (robot description, URDF)
Before this commit: robot allen_key_canonical, 1 links, 0 joints
Links:
- link object_root: mass 0.15 -> 0.045; geometry collision mesh filename=meshes/unit_hex_prism_x.obj scale=0.06 0.0057735 0.0057735; collision mesh filename=meshes/unit_hex_prism_x.obj scale=0.264 0.0057735 0.0057735

File: assets/urdf/workpieces/allen_key_hex_socket.urdf (robot description, URDF)
Before this commit: robot allen_key_hex_socket, 1 links, 0 joints
Links:
- link workpiece_root: geometry collision box size=0.008 0.020 0.025; collision box size=0.008 0.020 0.025

Commit message: Diversify Allen key adjustment grasps

File: assets/urdf/objects/allen_key_canonical.urdf (robot description, URDF)
Before this commit: robot allen_key_canonical, 1 links, 0 joints
Links:
- link object_root: mass 0.045 -> 0.060; geometry collision mesh filename=meshes/unit_hex_prism_x.obj scale=0.06 0.0057735 0.0057735; collision mesh filename=meshes/unit_hex_prism_x.obj scale=0.360 0.0057735 0.0057735

File: assets/urdf/table_allen_compact.urdf (robot description, URDF)
Before this commit: robot allen_compact_table, 1 links, 0 joints
Links:
- link box: geometry collision box size=0.16 0.14 0.12; visual box size=0.16 0.14 0.12

Commit message: Fixture lower Allen key workspace without table

File: assets/urdf/objects/allen_key_canonical.urdf (robot description, URDF)
Before this commit: robot allen_key_canonical, 1 links, 0 joints
Links:
- link object_root: mass 0.060 -> 0.045; geometry collision mesh filename=meshes/unit_hex_prism_x.obj scale=0.06 0.0057735 0.0057735; collision mesh filename=meshes/unit_hex_prism_x.obj scale=0.264 0.0057735 0.0057735
