Commit message: Enlarge Allen key turning table

File: assets/urdf/table_allen_turning.urdf (robot description, URDF)
Before this commit: robot allen_turning_table, 1 links, 0 joints
Links:
- link box: geometry collision box size=0.450 0.380 0.300; visual box size=0.450 0.380 0.300

Commit message: Fix resistance force

File: assets/urdf/table_allen_turning.urdf (robot description, URDF)
Before this commit: robot allen_turning_table, 1 links, 0 joints
Links:
- link box: geometry collision box size=0.600 0.350 0.300; visual box size=0.600 0.350 0.300
